File: photodiode.kicad_sch (KiCad schematic)
At the start: 4 parts

Commit message: solar panel init
Parts:
- D501: value D_Photo -> PDB-C160SM
Other:
- moved on the sheet: C501, C502, D501, R501
Changed lines of the file:
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@@
 (kicad_sch (version 20230121) (generator eeschema)
   (paper "A4")
-  (junction (at 135.89 115.57) (diameter 0) (color 0 0 0 0)
+  (junction (at 148.59 93.98) (diameter 0) (color 0 0 0 0)
   )
-  (junction (at 124.46 115.57) (diameter 0) (color 0 0 0 0)
+  (junction (at 137.16 93.98) (diameter 0) (color 0 0 0 0)
   )
-  (junction (at 135.89 123.19) (diameter 0) (color 0 0 0 0)
+  (junction (at 148.59 101.6) (diameter 0) (color 0 0 0 0)
   )
-  (junction (at 135.89 107.95) (diameter 0) (color 0 0 0 0)
+  (junction (at 148.59 86.36) (diameter 0) (color 0 0 0 0)
   )
-  (wire (pts (xy 135.89 123.19) (xy 135.89 124.46))
+  (wire (pts (xy 148.59 101.6) (xy 148.59 102.87))
     (stroke (width 0) (type default))
   )
-  (wire (pts (xy 124.46 107.95) (xy 135.89 107.95))
+  (wire (pts (xy 137.16 86.36) (xy 148.59 86.36))
     (stroke (width 0) (type default))
   )
-  (wire (pts (xy 135.89 115.57) (xy 151.13 115.57))
+  (wire (pts (xy 148.59 93.98) (xy 163.83 93.98))
     (stroke (width 0) (type default))
   )
-  (wire (pts (xy 124.46 115.57) (xy 135.89 115.57))
+  (wire (pts (xy 137.16 93.98) (xy 148.59 93.98))
     (stroke (width 0) (type default))
   )
-  (wire (pts (xy 135.89 106.68) (xy 135.89 107.95))
+  (wire (pts (xy 148.59 85.09) (xy 148.59 86.36))
     (stroke (width 0) (type default))
   )
-  (wire (pts (xy 124.46 123.19) (xy 135.89 123.19))
+  (wire (pts (xy 137.16 101.6) (xy 148.59 101.6))
     (stroke (width 0) (type default))
   )
   (text "I_sc = 80uA; I_dark = 2nA -> I_illum < 100uA\nV_photo = I_illum R <= 2.5 V -> R 25 kOhm"
-    (at 119.38 134.62 0)
+    (at 132.08 113.03 0)
     (effects (font (size 1.27 1.27)) (justify left bottom))
   )
-  (hierarchical_label "PHOTO_OUT" (shape output) (at 151.13 115.57 0) (fields_autoplaced)
+  (hierarchical_label "PHOTO_OUT" (shape output) (at 163.83 93.98 0) (fields_autoplaced)
     (effects (font (size 1.27 1.27)) (justify left))
   )
-  (symbol (lib_id "Device:C") (at 124.46 119.38 0) (unit 1)
+  (symbol (lib_id "Device:C") (at 137.16 97.79 0) (unit 1)
     (in_bom yes) (on_board yes) (dnp no) (fields_autoplaced)
-    (property "Reference" "C502" (at 127.381 118.7363 0)
+    (property "Reference" "C502" (at 140.081 97.1463 0)
       (effects (font (size 1.27 1.27)) (justify left))
     )
-    (property "Value" "100pF" (at 127.381 120.6573 0)
+    (property "Value" "100pF" (at 140.081 99.0673 0)
       (effects (font (size 1.27 1.27)) (justify left))
     )
-    (property "Footprint" "Capacitor_SMD:C_0603_1608Metric_Pad1.08x0.95mm_HandSolder" (at 125.4252 123.19 0)
+    (property "Footprint" "Capacitor_SMD:C_0603_1608Metric_Pad1.08x0.95mm_HandSolder" (at 138.1252 101.6 0)
       (effects (font (size 1.27 1.27)) hide)
     )
-    (property "Datasheet" "~" (at 124.46 119.38 0)
+    (property "Datasheet" "~" (at 137.16 97.79 0)
       (effects (font (size 1.27 1.27)) hide)
     )
@@
     )
   )
-  (symbol (lib_id "power:+3.3V") (at 135.89 106.68 0) (unit 1)
+  (symbol (lib_id "power:+3.3V") (at 148.59 85.09 0) (unit 1)
     (in_bom yes) (on_board yes) (dnp no) (fields_autoplaced)
-    (property "Reference" "#PWR0501" (at 135.89 110.49 0)
+    (property "Reference" "#PWR0501" (at 148.59 88.9 0)
       (effects (font (size 1.27 1.27)) hide)
     )
-    (property "Value" "+3.3V" (at 135.89 103.1781 0)
+    (property "Value" "+3.3V" (at 148.59 81.5881 0)
       (effects (font (size 1.27 1.27)))
     )
-    (property "Footprint" "" (at 135.89 106.68 0)
+    (property "Footprint" "" (at 148.59 85.09 0)
       (effects (font (size 1.27 1.27)) hide)
     )
-    (property "Datasheet" "" (at 135.89 106.68 0)
+    (property "Datasheet" "" (at 148.59 85.09 0)
       (effects (font (size 1.27 1.27)) hide)
     )
@@
     )
   )
-  (symbol (lib_id "Device:D_Photo") (at 135.89 113.03 270) (unit 1)
+  (symbol (lib_id "Device:D_Photo") (at 148.59 91.44 270) (unit 1)
     (in_bom yes) (on_board yes) (dnp no) (fields_autoplaced)
-    (property "Reference" "D501" (at 139.827 111.4338 90)
+    (property "Reference" "D501" (at 152.527 89.8438 90)
       (effects (font (size 1.27 1.27)) (justify left))
     )
-    (property "Value" "D_Photo" (at 139.827 113.3548 90)
+    (property "Value" "PDB-C160SM\n" (at 152.527 91.7648 90)
       (effects (font (size 1.27 1.27)) (justify left))
     )
-    (property "Footprint" "Diode_SMD:D_SMA_Handsoldering" (at 135.89 111.76 0)
+    (property "Footprint" "Diode_SMD:D_SMA_Handsoldering" (at 148.59 90.17 0)
       (effects (font (size 1.27 1.27)) hide)
     )
-    (property "Datasheet" "~" (at 135.89 111.76 0)
+    (property "Datasheet" "~" (at 148.59 90.17 0)
       (effects (font (size 1.27 1.27)) hide)
     )
@@
     )
   )
-  (symbol (lib_id "Device:R") (at 135.89 119.38 0) (unit 1)
+  (symbol (lib_id "Device:R") (at 148.59 97.79 0) (unit 1)
     (in_bom yes) (on_board yes) (dnp no) (fields_autoplaced)
-    (property "Reference" "R501" (at 137.668 118.7363 0)
+    (property "Reference" "R501" (at 150.368 97.1463 0)
       (effects (font (size 1.27 1.27)) (justify left))
     )
-    (property "Value" "24k 0.1%" (at 137.668 120.6573 0)
+    (property "Value" "24k 0.1%" (at 150.368 99.0673 0)
       (effects (font (size 1.27 1.27)) (justify left))
     )
-    (property "Footprint" "Resistor_SMD:R_0603_1608Metric_Pad0.98x0.95mm_HandSolder" (at 134.112 119.38 90)
+    (property "Footprint" "Resistor_SMD:R_0603_1608Metric_Pad0.98x0.95mm_HandSolder" (at 146.812 97.79 90)
       (effects (font (size 1.27 1.27)) hide)
     )
-    (property "Datasheet" "~" (at 135.89 119.38 0)
+    (property "Datasheet" "~" (at 148.59 97.79 0)
       (effects (font (size 1.27 1.27)) hide)
     )
@@
     )
   )
-  (symbol (lib_id "Device:C") (at 124.46 111.76 0) (unit 1)
+  (symbol (lib_id "Device:C") (at 137.16 90.17 0) (unit 1)
     (in_bom yes) (on_board yes) (dnp no) (fields_autoplaced)
-    (property "Reference" "C501" (at 127.381 111.1163 0)
+    (property "Reference" "C501" (at 140.081 89.5263 0)
       (effects (font (size 1.27 1.27)) (justify left))
     )
-    (property "Value" "0.1uF" (at 127.381 113.0373 0)
+    (property "Value" "0.1uF" (at 140.081 91.4473 0)
       (effects (font (size 1.27 1.27)) (justify left))
     )
-    (property "Footprint" "Capacitor_SMD:C_0603_1608Metric_Pad1.08x0.95mm_HandSolder" (at 125.4252 115.57 0)
+    (property "Footprint" "Capacitor_SMD:C_0603_1608Metric_Pad1.08x0.95mm_HandSolder" (at 138.1252 93.98 0)
       (effects (font (size 1.27 1.27)) hide)
     )
-    (property "Datasheet" "~" (at 124.46 111.76 0)
+    (property "Datasheet" "~" (at 137.16 90.17 0)
       (effects (font (size 1.27 1.27)) hide)
     )
@@
     )
   )
-  (symbol (lib_id "power:GND") (at 135.89 124.46 0) (unit 1)
+  (symbol (lib_id "power:GND") (at 148.59 102.87 0) (unit 1)
     (in_bom yes) (on_board yes) (dnp no) (fields_autoplaced)
-    (property "Reference" "#PWR0502" (at 135.89 130.81 0)
+    (property "Reference" "#PWR0502" (at 148.59 109.22 0)
       (effects (font (size 1.27 1.27)) hide)
     )
-    (property "Value" "GND" (at 135.89 128.5955 0)
+    (property "Value" "GND" (at 148.59 107.0055 0)
       (effects (font (size 1.27 1.27)))
     )
-    (property "Footprint" "" (at 135.89 124.46 0)
+    (property "Footprint" "" (at 148.59 102.87 0)
       (effects (font (size 1.27 1.27)) hide)
     )
-    (property "Datasheet" "" (at 135.89 124.46 0)
+    (property "Datasheet" "" (at 148.59 102.87 0)
       (effects (font (size 1.27 1.27)) hide)
     )
