File: pv_cells.kicad_sch (KiCad schematic)
At the start: 9 parts

Commit message: rev 1.0, added pdf
Parts:
- D601, D602, D603: footprint TO254P1524X483-4N -> SamacSys_Parts:TO254P1524X483-4N
- SC601, SC602, SC603, SC604, SC605, SC606: footprint (none) -> Solar_cell:XTJPrime_solar_cell
Changed lines of the file:
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@@
       (effects (font (size 1.27 1.27)) (justify right))
     )
-    (property "Footprint" "TO254P1524X483-4N" (at 209.22 69.85 0)
+    (property "Footprint" "SamacSys_Parts:TO254P1524X483-4N" (at 209.22 69.85 0)
       (effects (font (size 1.27 1.27)) (justify left top) hide)
     )
@@
       (effects (font (size 1.27 1.27)) (justify left))
     )
-    (property "Footprint" "" (at 138.43 112.776 90)
+    (property "Footprint" "Solar_cell:XTJPrime_solar_cell" (at 138.43 112.776 90)
       (effects (font (size 1.27 1.27)) hide)
     )
@@
       (effects (font (size 1.27 1.27)) (justify left))
     )
-    (property "Footprint" "" (at 160.02 125.476 90)
+    (property "Footprint" "Solar_cell:XTJPrime_solar_cell" (at 160.02 125.476 90)
       (effects (font (size 1.27 1.27)) hide)
     )
@@
       (effects (font (size 1.27 1.27)) (justify left))
     )
-    (property "Footprint" "" (at 160.02 112.776 90)
+    (property "Footprint" "Solar_cell:XTJPrime_solar_cell" (at 160.02 112.776 90)
       (effects (font (size 1.27 1.27)) hide)
     )
@@
       (effects (font (size 1.27 1.27)) (justify left))
     )
-    (property "Footprint" "" (at 138.43 125.476 90)
+    (property "Footprint" "Solar_cell:XTJPrime_solar_cell" (at 138.43 125.476 90)
       (effects (font (size 1.27 1.27)) hide)
     )
@@
       (effects (font (size 1.27 1.27)) (justify right))
     )
-    (property "Footprint" "TO254P1524X483-4N" (at 254.94 69.85 0)
+    (property "Footprint" "SamacSys_Parts:TO254P1524X483-4N" (at 254.94 69.85 0)
       (effects (font (size 1.27 1.27)) (justify left top) hide)
     )
@@
       (effects (font (size 1.27 1.27)) (justify left))
     )
-    (property "Footprint" "" (at 116.84 125.476 90)
+    (property "Footprint" "Solar_cell:XTJPrime_solar_cell" (at 116.84 125.476 90)
       (effects (font (size 1.27 1.27)) hide)
     )
@@
       (effects (font (size 1.27 1.27)))
     )
-    (property "Footprint" "" (at 116.84 112.776 90)
+    (property "Footprint" "Solar_cell:XTJPrime_solar_cell" (at 116.84 112.776 90)
       (effects (font (size 1.27 1.27)) hide)
     )
@@
       (effects (font (size 1.27 1.27)) (justify right))
     )
-    (property "Footprint" "TO254P1524X483-4N" (at 233.35 69.85 0)
-      (effects (font (size 1.27 1.27)) (justify left top) hide)
-    )
+    (property "Footprint" "SamacSys_Parts:TO254P1524X483-4N" (at 233.35 69.85 0)
+      (effects (font (size 1.27 1.27)) (justify left top) hide)
+    )

Commit message: rev 1.0 routed by Jonah
Connections:
- net PV_V- renamed GND
Changed lines of the file:
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@@
-    (stroke (width 0) (type default))
-  )
-  (wire (pts (xy 138.43 138.43) (xy 176.53 138.43))
     (stroke (width 0) (type default))
   )
@@
     (effects (font (size 1.27 1.27)) (justify left))
   )
-  (hierarchical_label "PV_V-" (shape input) (at 176.53 138.43 0) (fields_autoplaced)
-    (effects (font (size 1.27 1.27)) (justify left))
+  (netclass_flag "" (length 2.54) (shape dot) (at 160.02 119.38 270) (fields_autoplaced)
+    (effects (font (size 1.27 1.27)) (justify right bottom))
+    (property "Netclass" "RawPower" (at 162.56 118.6815 90)
+      (effects (font (size 1.27 1.27) italic) (justify left) hide)
+    )
+  )
+  (netclass_flag "" (length 2.54) (shape dot) (at 116.84 119.38 270) (fields_autoplaced)
+    (effects (font (size 1.27 1.27)) (justify right bottom))
+    (property "Netclass" "RawPower" (at 119.38 118.6815 90)
+      (effects (font (size 1.27 1.27) italic) (justify left) hide)
+    )
+  )
+  (netclass_flag "" (length 2.54) (shape dot) (at 116.84 106.68 270) (fields_autoplaced)
+    (effects (font (size 1.27 1.27)) (justify right bottom))
+    (property "Netclass" "RawPower" (at 119.38 105.9815 90)
+      (effects (font (size 1.27 1.27) italic) (justify left) hide)
+    )
+  )
+  (netclass_flag "" (length 2.54) (shape dot) (at 138.43 106.68 90) (fields_autoplaced)
+    (effects (font (size 1.27 1.27)) (justify left bottom))
+    (property "Netclass" "RawPower" (at 135.89 105.9815 90)
+      (effects (font (size 1.27 1.27) italic) (justify left) hide)
+    )
+  )
+  (netclass_flag "" (length 2.54) (shape dot) (at 138.43 119.38 270) (fields_autoplaced)
+    (effects (font (size 1.27 1.27)) (justify right bottom))
+    (property "Netclass" "RawPower" (at 140.97 118.6815 90)
+      (effects (font (size 1.27 1.27) italic) (justify left) hide)
+    )
+  )
+  (netclass_flag "" (length 2.54) (shape dot) (at 160.02 106.68 90) (fields_autoplaced)
+    (effects (font (size 1.27 1.27)) (justify left bottom))
+    (property "Netclass" "RawPower" (at 157.48 105.9815 90)
+      (effects (font (size 1.27 1.27) italic) (justify left) hide)
+    )
   )
   (symbol (lib_id "SamacSys_Parts:SM74611KTTR") (at 114.3 106.68 90) (unit 1)
@@
         )
       )
+    )
+  )
+  (symbol (lib_id "power:GND") (at 138.43 138.43 0) (unit 1)
+    (in_bom yes) (on_board yes) (dnp no) (fields_autoplaced)
+    (property "Reference" "#PWR0601" (at 138.43 144.78 0)
+      (effects (font (size 1.27 1.27)) hide)
+    )
+    (property "Value" "GND" (at 138.43 142.5655 0)
+      (effects (font (size 1.27 1.27)))
+    )
+    (property "Footprint" "" (at 138.43 138.43 0)
+      (effects (font (size 1.27 1.27)) hide)
+    )
+    (property "Datasheet" "" (at 138.43 138.43 0)
+      (effects (font (size 1.27 1.27)) hide)
+    )
+    (pin "1")
+    (instances
+      (project "solar-panel"
+        (path "/3cfd2153-52bb-4eed-95c6-13d99c50d08a/6b0b648d-c14f-4b9c-9278-56619c685686"
+          (reference "#PWR0601") (unit 1)
+        )
+      )
