File: solar-panel.kicad_pcb (KiCad board)
At the start: 2 copper layers, 320 x 82 mm, 35 parts, among them J101 Conn_01x05_Pin, J102 Conn_01x02, U101 MCP3008, U201 SS39ET, U301 LMT87DCK, U401 LMT87DCK

Commit message: Remade schematic for all panels Fixed lightricity footprint Erased panel PCBs
Parts:
- removed C101, C201, C301, C401, C501: 0.1uF, Capacitor_SMD:C_0603_1608Metric_Pad1.08x0.95mm_HandSolder
- removed C502: 100pF, Capacitor_SMD:C_0603_1608Metric_Pad1.08x0.95mm_HandSolder
- removed D501: PDB-C160SM, Diode_SMD:D_SMA_Handsoldering
- removed D601, D602, D603: SM74611KTTR, SamacSys_Parts:TO254P1524X483-4N
- removed G*** (x2): LOGO, USST_logo:lightning_bolt
- removed G***: LOGO, USST_logo:usask_logo_20x4
- removed G***: LOGO, USST_logo:u_of_r_logo_20x8
- removed G***: LOGO, USST_logo:USST_logo
- removed H101, H102, H103, H104, H105, H106: MountingHole, MountingHole:MountingHole_2.7mm
- removed J101: Conn_01x05_Pin, Connector_Hirose:Hirose_DF13-05P-1.25DSA_1x05_P1.25mm_Vertical
- removed J102: Conn_01x02, Connector_PinHeader_2.54mm:PinHeader_1x02_P2.54mm_Vertical
- removed R501: 24k 0.1%, Resistor_SMD:R_0603_1608Metric_Pad0.98x0.95mm_HandSolder
- removed REF**: ESD-Logo_8.9x8mm_SilkScreen, Symbol:ESD-Logo_8.9x8mm_SilkScreen
- removed SC601, SC602, SC603, SC604, SC605, SC606: XTJPrime, Solar_cell:XTJPrime_solar_cell
- removed U101: MCP3008, Package_SO:SOIC-16_3.9x9.9mm_P1.27mm
- removed U201: SS39ET, SamacSys_Parts:SOT95P280X140-3N
- removed U301, U401: LMT87DCK, Package_TO_SOT_SMD:SOT-353_SC-70-5
Routing:
- net /Solar Cells/PV_V+: track 241.2 -> 0.00 mm, vias 3 -> 0
- net GND: track 133.6 -> 0.00 mm, vias 1 -> 0
- net +3.3V: track 131.1 -> 0.00 mm
- net Net-(SC601--): track 128.7 -> 0.00 mm
- net Net-(SC605--): track 127.2 -> 0.00 mm
- net Net-(SC603--): track 124.7 -> 0.00 mm
- net Net-(D601-ANODE_1): track 85.8 -> 0.00 mm
- net Net-(D603-ANODE_1): track 84.9 -> 0.00 mm
- net /Sun sensor/PHOTO_OUT: track 78.7 -> 0.00 mm
- net Net-(D602-ANODE_1): track 76.1 -> 0.00 mm
- net /Mag Sensor/MAG_OUT: track 71.9 -> 0.00 mm
- net /Temp Sensor 2/TEMP_OUT: track 71.7 -> 0.00 mm
- net /SCK: track 14.1 -> 0.00 mm
- net /MISO: track 14.0 -> 0.00 mm
- net /MOSI: track 13.8 -> 0.00 mm
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- added copper zone on B.Cu, net (none)
- added copper zone on F.Cu, net (none)
- removed copper zone on B.Cu, net GND
- removed copper zone on F.Cu, net GND
Other:
- board text removed: "May 27, 2023"
- board text removed: "SCH: Atharva K. LAYOUT: Jonah R."
- board text removed: "Solar Panels Rev 1.0"
- board text removed: "{dblquote}Caps, Diodes and Hope.{dblquote}"

Commit message: rearanged panels, updated solar cells footprint
Parts:
- added H101: MountingHole, MountingHole:MountingHole_2.7mm, F.Cu at (75.0, 278.7)
- added H102: MountingHole, MountingHole:MountingHole_2.7mm, F.Cu at (75.0, 285.7)
- added H103: MountingHole, MountingHole:MountingHole_2.7mm, F.Cu at (82.0, 278.7)
- added H104: MountingHole, MountingHole:MountingHole_2.7mm, F.Cu at (82.0, 285.7)
- added H105: MountingHole, MountingHole:MountingHole_2.7mm, F.Cu at (88.9, 278.7)
- added H106: MountingHole, MountingHole:MountingHole_2.7mm, F.Cu at (88.9, 285.7)
- added J1: Conn_01x02_Pin, Connector_PinSocket_2.54mm:PinSocket_1x02_P2.54mm_Vertical, F.Cu at (46.3, 277.6)
- added J2: Conn_01x02_Pin, Connector_PinSocket_2.54mm:PinSocket_1x02_P2.54mm_Vertical, F.Cu at (50.9, 277.6)
- added J3: Conn_01x02_Pin, Connector_PinSocket_2.54mm:PinSocket_1x02_P2.54mm_Vertical, F.Cu at (55.5, 277.6)
- added J4: Conn_01x02_Pin, Connector_PinSocket_2.54mm:PinSocket_1x02_P2.54mm_Vertical, F.Cu at (60.1, 277.6)
- added J5: Conn_01x02_Pin, Connector_PinSocket_2.54mm:PinSocket_1x02_P2.54mm_Vertical, F.Cu at (64.7, 277.6)
- added J6: Conn_01x02_Pin, Connector_PinSocket_2.54mm:PinSocket_1x02_P2.54mm_Vertical, F.Cu at (69.3, 277.6)
- added SC1: S8040_CIC, Solar_cell:Solar_Cell_Lightricity_S8040_CIC, F.Cu at (58.5, 95.5)
- added SC10: S8040_CIC, Solar_cell:Solar_Cell_Lightricity_S8040_CIC, F.Cu at (136.5, 187.5)
- added SC11: S8040_CIC, Solar_cell:Solar_Cell_Lightricity_S8040_CIC, F.Cu at (58.5, 279.5)
- added SC12: S8040_CIC, Solar_cell:Solar_Cell_Lightricity_S8040_CIC, F.Cu at (108.5, 279.5)
- added SC13: S8040_CIC, Solar_cell:Solar_Cell_Lightricity_S8040_CIC, F.Cu at (158.5, 279.5)
- added SC14: S8040_CIC, Solar_cell:Solar_Cell_Lightricity_S8040_CIC, F.Cu at (208.5, 279.5)
- added SC15: S8040_CIC, Solar_cell:Solar_Cell_Lightricity_S8040_CIC, F.Cu at (258.5, 279.5)
- added SC2: S8040_CIC, Solar_cell:Solar_Cell_Lightricity_S8040_CIC, F.Cu at (108.5, 95.5)
- added SC3: S8040_CIC, Solar_cell:Solar_Cell_Lightricity_S8040_CIC, F.Cu at (158.5, 95.6)
- added SC4: S8040_CIC, Solar_cell:Solar_Cell_Lightricity_S8040_CIC, F.Cu at (208.5, 95.6)
- added SC5: S8040_CIC, Solar_cell:Solar_Cell_Lightricity_S8040_CIC, F.Cu at (258.5, 95.6)
- added SC6: S8040_CIC, Solar_cell:Solar_Cell_Lightricity_S8040_CIC, F.Cu at (247.5, 187.5)
- added SC7: S8040_CIC, Solar_cell:Solar_Cell_Lightricity_S8040_CIC, F.Cu at (297.5, 187.5)
- added SC8: S8040_CIC, Solar_cell:Solar_Cell_Lightricity_S8040_CIC, F.Cu at (36.5, 187.5)
- added SC9: S8040_CIC, Solar_cell:Solar_Cell_Lightricity_S8040_CIC, F.Cu at (86.5, 187.5)
Routing:
- removed copper zone on B.Cu, net (none)
- removed copper zone on F.Cu, net (none)
Other:
- board size 320 x 82 mm -> 312 x 268.5 mm

Commit message: Added traces, added solder pads for connections (NO GND PADS)
Parts:
- removed J1, J2, J3, J4, J5, J6: Conn_01x02_Pin, Connector_PinSocket_2.54mm:PinSocket_1x02_P2.54mm_Vertical
- added REF**: Series_Connection_Pad, Connection_Pads:Series_Connection_Pad, F.Cu at (712.5, 263.0)
- added REF**: Series_Connection_Pad, Connection_Pads:Series_Connection_Pad, F.Cu at (801.0, 123.6)
- added REF**: Series_Connection_Pad, Connection_Pads:Series_Connection_Pad, F.Cu at (730.0, 261.5)
- added REF**: Series_Connection_Pad, Connection_Pads:Series_Connection_Pad, F.Cu at (823.0, 51.0)
- added REF**: Series_Connection_Pad, Connection_Pads:Series_Connection_Pad, F.Cu at (731.5, 163.5)
- added REF**: Series_Connection_Pad, Connection_Pads:Series_Connection_Pad, F.Cu at (825.5, 131.0)
- added SC12: S8040_CIC, Solar_cell:Solar_Cell_Lightricity_S8040_CIC, F.Cu at (724.0, 25.5)
- moved SC11 837.5 mm to (896.0, 273.0), turned to 90 degrees
- moved SC12 789.5 mm to (896.0, 223.0), turned to 90 degrees
- moved SC13 745.1 mm to (896.0, 173.0), turned to 90 degrees
- moved SC14 705.1 mm to (896.0, 123.0), turned to 90 degrees
- moved SC8 689.1 mm to (725.5, 177.0), turned to -90 degrees
- moved SC1 677.2 mm to (712.0, 273.0), turned to 90 degrees
- moved SC15 670.1 mm to (896.0, 73.0), turned to 90 degrees
- moved SC9 640.2 mm to (725.5, 227.0), turned to -90 degrees
- moved SC2 616.8 mm to (712.0, 223.0), turned to 90 degrees
- moved SC10 595.8 mm to (725.5, 277.0), turned to -90 degrees
- moved SC3 559.0 mm to (712.1, 173.0), turned to 90 degrees
- moved SC4 504.3 mm to (712.1, 123.0), turned to 90 degrees
- moved SC6 489.1 mm to (724.0, 77.0), turned to -90 degrees
- moved SC5 454.1 mm to (712.1, 73.0), turned to 90 degrees
- moved SC7 430.8 mm to (724.0, 127.0), turned to -90 degrees
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- renumbered H101 to H1, H104 to H2, H102 to H3, H105 to H4, H103 to H5, H106 to H6
Connections:
- SC1 pad 1: Net-(J2-Pin_2) -> unconnected-(SC1-+-Pad1)
- SC10 pad 2: Net-(J5-Pin_1) -> unconnected-(SC10---Pad2)
- SC11 pad 1: Net-(J1-Pin_1) -> unconnected-(SC11-+-Pad1)
- SC15 pad 2: Net-(J1-Pin_2) -> GND
- SC5 pad 2: Net-(J2-Pin_1) -> GND
- SC6 pad 1: Net-(J3-Pin_2) -> unconnected-(SC6-+-Pad1)
- SC7 pad 2: Net-(J2-Pin_2) -> unconnected-(SC7---Pad2)
- SC8 pad 1: Net-(J6-Pin_2) -> unconnected-(SC8-+-Pad1)
Routing:
- net unconnected-(SC11-+-Pad1): track 0.00 -> 187.3 mm, vias 0 -> 1
- net Net-(SC12--): track 0.00 -> 144.5 mm
- net Net-(SC8--): track 0.00 -> 126.2 mm
- net Net-(SC2--): track 0.00 -> 111.3 mm
- net Net-(SC4--): track 0.00 -> 111.2 mm
- net Net-(SC11--): track 0.00 -> 111.2 mm
- net Net-(SC6--): track 0.00 -> 111.2 mm
- net Net-(SC14--): track 0.00 -> 111.2 mm
- net Net-(SC1--): track 0.00 -> 111.2 mm
- net Net-(SC3--): track 0.00 -> 111.2 mm
- net Net-(SC10-+): track 0.00 -> 110.6 mm
- net Net-(SC13--): track 0.00 -> 110.4 mm
- net unconnected-(SC10---Pad2): track 0.00 -> 108.3 mm, vias 0 -> 1
- net unconnected-(SC6-+-Pad1): track 0.00 -> 106.9 mm, vias 0 -> 1
- net unconnected-(SC7---Pad2): track 0.00 -> 80.3 mm
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- added copper zone on F.Cu, net GND
Other:
- board size 312 x 268.5 mm -> 268.5 x 326 mm

Commit message: Replace solder pads with hirose df13 connections
Parts:
- removed REF** (x6): Series_Connection_Pad, Connection_Pads:Series_Connection_Pad
- removed the SC12 at (724.0, 25.5)
- added Buck_1: ~, Connection_Pads:2_Hirose_Pin, F.Cu at (734.4, 113.4)
- added Buck_2A1: ~, Connection_Pads:2_Hirose_Pin, F.Cu at (702.4, 164.1)
- added Buck_2B1: ~, Connection_Pads:2_Hirose_Pin, F.Cu at (815.4, 127.1)
- added Sepic_A1: ~, Connection_Pads:2_Hirose_Pin, F.Cu at (700.6, 269.8)
- added Sepic_B1: ~, Connection_Pads:2_Hirose_Pin, F.Cu at (828.6, 254.9)
- moved H6 0.33 mm to (367.0, 246.0)
- renumbered SC9 to SC10, SC10 to SC11, SC11 to SC2, SC2 to SC3, SC3 to SC4, SC4 to SC5, SC5 to SC6, SC6 to SC7, SC7 to SC8, SC8 to SC9
Connections:
- SC1 pad 1: unconnected-(SC1-+-Pad1) -> Net-(SC1-+)
- SC11 pad 2: unconnected-(SC10---Pad2) -> Net-(Buck_1-BCR-)
- SC12 pad 1: Net-(SC11--) -> Net-(Buck_2B1-BCR+)
- SC15 pad 2: GND -> Net-(Buck_2B1-BCR-)
- SC2 pad 1: unconnected-(SC11-+-Pad1) -> Net-(SC2-+)
- SC2 pad 2: Net-(SC11--) -> Net-(SC2--)
- SC3 pad 1: Net-(SC1--) -> Net-(Buck_2A1-BCR+)
- SC6 pad 2: GND -> Net-(Buck_2A1-BCR-)
- SC7 pad 1: unconnected-(SC6-+-Pad1) -> Net-(Buck_1-BCR+)
- SC8 pad 2: unconnected-(SC7---Pad2) -> Net-(SC8--)
- SC9 pad 1: unconnected-(SC8-+-Pad1) -> Net-(SC8--)
Routing:
- net Net-(Buck_1-BCR-): track 0.00 -> 280.4 mm, vias 0 -> 1
- net Net-(Buck_2A1-BCR-): track 0.00 -> 206.6 mm, vias 0 -> 1
- net unconnected-(SC11-+-Pad1): track 187.3 -> 0.00 mm, vias 1 -> 0
- net Net-(Buck_2B1-BCR+): track 0.00 -> 142.7 mm, vias 0 -> 1
- net Net-(Buck_2B1-BCR-): track 0.00 -> 132.7 mm, vias 0 -> 1
- net Net-(SC8--): track 0.00 -> 121.8 mm
- net Net-(Buck_2A1-BCR+): track 0.00 -> 114.8 mm, vias 0 -> 1
- net Net-(SC11--): track 111.2 -> 0.00 mm
- net unconnected-(SC10---Pad2): track 108.3 -> 0.00 mm, vias 1 -> 0
- net unconnected-(SC6-+-Pad1): track 106.9 -> 0.00 mm, vias 1 -> 0
- net Net-(Buck_1-BCR+): track 0.00 -> 103.7 mm, vias 0 -> 1
- net unconnected-(SC7---Pad2): track 80.3 -> 0.00 mm
- net unconnected-(SC15---Pad2): track 79.6 -> 0.00 mm, vias 1 -> 0
- net Net-(SC2-+): track 0.00 -> 79.4 mm, vias 0 -> 1
- net Net-(SC2--): track 0.00 -> 78.5 mm, vias 0 -> 1
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- removed copper zone on F.Cu, net GND
Other:
- board size 268.5 x 326 mm -> 268.5 x 287 mm

Commit message: Added Mounting holes, overlapped cells, changed to 5 6 3 configuration, changed overall solar panel dimensions
Parts:
- removed Buck_1, Buck_2A1, Buck_2B1, Sepic_A1, Sepic_B1: ~, Connection_Pads:2_Hirose_Pin
- removed SC15: S8040_CIC, Solar_cell:Solar_Cell_Lightricity_S8040_CIC
- added Buck1: ~, Connection_Pads:2_Hirose_Pin, B.Cu at (712.8, 174.7)
- added Buck2: ~, Connection_Pads:2_Hirose_Pin, B.Cu at (722.6, 228.9)
- added H1: MountingHole, MountingHole:MountingHole_2.7mm, F.Cu at (585.0, 253.5)
- added H1: MountingHole, MountingHole:MountingHole_2.7mm, F.Cu at (728.0, 279.5)
- added H10: MountingHole, MountingHole:MountingHole_2.7mm, F.Cu at (585.0, 261.5)
- added H2: MountingHole, MountingHole:MountingHole_2.7mm, F.Cu at (806.5, 142.0)
- added H2: MountingHole, MountingHole:MountingHole_2.7mm, F.Cu at (806.5, 42.5)
- added H4: MountingHole, MountingHole:MountingHole_2.7mm, F.Cu at (727.0, 43.5)
- added H7: MountingHole, MountingHole:MountingHole_2.7mm, F.Cu at (585.0, 269.8)
- added H8: MountingHole, MountingHole:MountingHole_2.7mm, F.Cu at (585.0, 276.8)
- added H9: MountingHole, MountingHole:MountingHole_2.7mm, F.Cu at (585.0, 283.7)
- added Sepic1: ~, Connection_Pads:2_Hirose_Pin, B.Cu at (820.1, 179.3)
- moved H2 505.1 mm to (805.5, 3.00)
- moved H1 450.4 mm to (806.0, 321.0)
- moved H5 445.1 mm to (728.0, 3.10)
- moved H6 375.5 mm to (728.0, 142.5)
- moved H3 365.9 mm to (727.5, 321.0)
- moved H4 226.8 mm to (586.5, 246.5)
- moved SC14 185.3 mm to (723.9, 54.2), turned to -90 degrees
- moved SC2 166.4 mm to (822.2, 123.8), turned to -90 degrees
- moved SC13 101.2 mm to (822.0, 242.0), turned to -90 degrees
- moved SC12 88.1 mm to (822.1, 174.9), turned to -90 degrees
- moved SC8 20.0 mm to (724.0, 147.0)
- moved SC7 19.3 mm to (723.9, 96.2)
- moved SC9 12.9 mm to (723.9, 189.8)
- moved SC5 11.7 mm to (710.1, 134.6)
- moved SC10 7.40 mm to (724.0, 234.2)
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Connections:
- SC12 pad 1: Net-(Buck_2B1-BCR+) -> Net-(SC12-+)
- SC14 pad 1: Net-(SC13--) -> Net-(Buck2-BCR+)
- SC2 pad 2: Net-(SC2--) -> Net-(SC12-+)
- SC3 pad 1: Net-(Buck_2A1-BCR+) -> Net-(SC1--)
- SC7 pad 1: Net-(Buck_1-BCR+) -> Net-(SC14--)
Routing:
- net Net-(Buck2-BCR+): track 0.00 -> 221.8 mm, vias 0 -> 1
- net Net-(Buck_2B1-BCR+): track 142.7 -> 0.00 mm, vias 1 -> 0
- net Net-(Buck2-BCR-): track 280.4 -> 139.9 mm
- net Net-(Buck_2B1-BCR-): track 132.7 -> 0.00 mm, vias 1 -> 0
- net Net-(Buck_2A1-BCR+): track 114.8 -> 0.00 mm, vias 1 -> 0
- net Net-(SC12-+): track 0.00 -> 114.6 mm
- net Net-(Buck_1-BCR+): track 103.7 -> 0.00 mm, vias 1 -> 0
- net Net-(Buck1-BCR+): track 59.5 -> 152.2 mm
- net Net-(SC2--): track 78.5 -> 0.00 mm, vias 1 -> 0
- net Net-(SC13--): track 110.4 -> 148.3 mm, vias 0 -> 1
- net Net-(SC2-+): track 79.4 -> 111.5 mm
- net Net-(SC10-+): track 135.9 -> 104.1 mm
- net Net-(SC1--): track 96.6 -> 122.8 mm, vias 1 -> 0
- net Net-(SC12--): track 111.7 -> 136.4 mm
- net Net-(SC7--): track 111.7 -> 132.1 mm
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Other:
- board size 268.5 x 287 mm -> 275.4 x 326.4 mm

Commit message: Updated footprint to match new knowledge of bypass diodes
Parts:
- moved Buck2 161.4 mm to (741.6, 68.6), turned to 0 degrees
- moved Sepic1 104.7 mm to (816.6, 74.7)
- moved Buck1 98.7 mm to (703.4, 76.4), turned to -90 degrees
- moved H2 4.84 mm to (806.8, 37.7)
- moved SC9 4.68 mm to (724.7, 194.4)
- moved SC14 1.99 mm to (724.4, 52.3)
- moved SC7 1.93 mm to (724.2, 94.3)
- moved SC8 1.93 mm to (725.2, 148.5)
- moved SC10 1.87 mm to (724.3, 236.1)
- moved SC3 0.97 mm to (710.1, 218.7)
- moved SC11 0.64 mm to (724.4, 277.5)
Routing:
- net Net-(Buck2-BCR+): track 221.8 -> 0.00 mm, vias 1 -> 0
- net Net-(Buck1-BCR-): track 201.2 -> 0.00 mm, vias 1 -> 0
- net Net-(Buck1-BCR+): track 152.2 -> 0.00 mm, vias 1 -> 0
- net Net-(SC13--): track 148.3 -> 0.00 mm, vias 1 -> 0
- net Net-(Buck2-BCR-): track 139.9 -> 0.00 mm, vias 1 -> 0
- net Net-(SC12--): track 136.4 -> 0.00 mm
- net Net-(SC7--): track 132.1 -> 0.00 mm
- net Net-(SC5--): track 128.8 -> 0.00 mm
- net Net-(SC1--): track 122.8 -> 0.00 mm
- net Net-(SC3--): track 117.4 -> 0.00 mm
- net Net-(SC12-+): track 114.6 -> 0.00 mm
- net Net-(SC2-+): track 111.5 -> 0.00 mm, vias 1 -> 0
- net Net-(SC4--): track 101.9 -> 0.00 mm
- net Net-(SC14--): track 101.6 -> 0.00 mm
- net Net-(SC10--): track 103.8 -> 58.5 mm
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Other:
- outline, holes or cut-outs redrawn

Commit message: made projects for manufacturing each individual solar panel
Parts:
- moved H4 628.5 mm to (1215.0, 251.3)
- moved H2 599.7 mm to (1384.7, 301.3)
- moved SC10 580.4 mm to (1304.1, 211.0)
- moved SC9 580.0 mm to (1304.2, 169.8)
- moved SC11 580.0 mm to (1304.0, 257.7)
- moved SC7 579.7 mm to (1303.8, 81.3)
- moved SC14 579.7 mm to (1303.9, 39.3)
- moved SC8 579.3 mm to (1304.1, 128.5)
- moved H2 578.5 mm to (1384.6, 9.79)
- moved Buck2 576.1 mm to (1317.6, 58.8)
- moved H4 444.9 mm to (1171.1, 17.6)
- moved H3 443.8 mm to (1171.1, 309.1)
- moved H1 443.4 mm to (1171.1, 264.1)
- moved H5 443.3 mm to (1171.1, -9.44)
- moved H6 443.2 mm to (1171.1, 135.6)
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Routing:
- net Net-(SC8--): track 78.6 -> 0.00 mm
- net Net-(SC10-+): track 72.6 -> 0.00 mm
- net Net-(SC10--): track 58.5 -> 0.00 mm
Other:
- board size 275.4 x 326.4 mm -> 761.4 x 326.5 mm
