File: left-panel/left-panel/left-panel.kicad_pcb (KiCad board)
At the start: 2 copper layers, 84.7 x 251 mm, 17 parts

Commit message: Added projects for blank PCBs, updated solar panels
Parts:
- removed the H1 at (566.5, 234.1)
- removed H2, H3: MountingHole, MountingHole:MountingHole_2.7mm
- moved H1 301.8 mm to (832.2, 80.4)
- moved H4 294.7 mm to (832.2, 99.9)
- moved H6 284.9 mm to (822.2, 90.3)
- moved H5 276.5 mm to (822.2, 99.9)
- moved H9 249.8 mm to (832.2, 247.9)
- moved H10 249.4 mm to (832.2, 228.4)
- moved H7 239.2 mm to (822.2, 238.4)
- moved H8 238.9 mm to (822.2, 247.9)
- moved SC1 127.6 mm to (836.4, 295.4)
- moved SC5 126.2 mm to (836.2, 144.5)
- moved SC4 126.2 mm to (836.1, 186.1)
- moved SC3 125.9 mm to (835.8, 227.5)
- moved SC6 125.0 mm to (835.3, 78.5)
- moved Buck1 110.9 mm to (826.9, 68.1), turned to -90 degrees
Routing:
- net Net-(Buck1-BCR+): track 0.00 -> 336.4 mm, vias 0 -> 1
- net Net-(SC1--): track 0.00 -> 114.0 mm
- net Net-(SC5--): track 0.00 -> 96.8 mm
- net Net-(SC3--): track 0.00 -> 72.7 mm
- net Net-(SC4--): track 0.00 -> 55.0 mm
- net Net-(Buck1-BCR-): track 0.00 -> 43.5 mm, vias 0 -> 1
Other:
- board size 84.7 x 251 mm -> 85 x 270 mm
