File: right-panel/right-panel/right-panel.kicad_pcb (KiCad board)
At the start: 2 copper layers, 84.5 x 251 mm, 4 parts

Commit message: Added projects for blank PCBs, updated solar panels
Parts:
- added H1: MountingHole, MountingHole:MountingHole_2.7mm, F.Cu at (940.8, 222.2)
- added H2: MountingHole, MountingHole:MountingHole_2.7mm, F.Cu at (950.8, 231.8)
- added H3: MountingHole, MountingHole:MountingHole_2.7mm, F.Cu at (940.8, 241.7)
- added H4: MountingHole, MountingHole:MountingHole_2.7mm, F.Cu at (950.8, 83.8)
- added H5: MountingHole, MountingHole:MountingHole_2.7mm, F.Cu at (940.8, 93.8)
- added H6: MountingHole, MountingHole:MountingHole_2.7mm, F.Cu at (950.8, 222.2)
- added H7: MountingHole, MountingHole:MountingHole_2.7mm, F.Cu at (940.8, 74.3)
- added H8: MountingHole, MountingHole:MountingHole_2.7mm, F.Cu at (950.8, 74.3)
- moved Sepic1 133.3 mm to (950.5, 49.9), turned to 90 degrees
- moved SC13 115.4 mm to (936.4, 256.3)
- moved SC2 114.7 mm to (936.8, 122.1)
- moved SC12 114.4 mm to (936.5, 173.7)
Routing:
- net Net-(SC13--): track 0.00 -> 274.3 mm, vias 0 -> 1
- net Net-(SC2-+): track 0.00 -> 133.9 mm, vias 0 -> 1
- net Net-(SC12--): track 0.00 -> 113.8 mm
- net Net-(SC12-+): track 0.00 -> 103.3 mm
Other:
- board size 84.5 x 251 mm -> 85 x 270 mm
