File: -x_panel/-x_panel/right-panel.kicad_sch (KiCad schematic)
At the start: 15 parts

Commit message: Changes solar panels
Parts:
- SC2: footprint Solar_cell:Solar_Cell_Lightricity_S8040_CIC -> Solar_cell:Solar_Cell_Lightricity_S8040_CIC_Shorter_Tabs
- Sepic1: footprint Connection_Pads:2_Hirose_Pin -> Connection_Pads:DF13_Horizontal
Changed lines of the file:
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@@
 			)
 		)
-		(property "Footprint" "Solar_cell:Solar_Cell_Lightricity_S8040_CIC"
+		(property "Footprint" "Solar_cell:Solar_Cell_Lightricity_S8040_CIC_Shorter_Tabs"
 			(at 149.86 63.246 90)
 			(effects
@@
 			)
 		)
-		(property "Footprint" "Connection_Pads:2_Hirose_Pin"
+		(property "Footprint" "Connection_Pads:DF13_Horizontal"
 			(at 139.7 55.88 0)
 			(effects
