File: +x_panel/left-panel/left-panel.kicad_sch (KiCad schematic)
At the start: 21 parts

Commit message: Updated panels based on dxf drawings from mech, need to move all holes up 5mm
Parts:
- SC3: footprint Solar_cell:Solar_Cell_Lightricity_S8040_CIC -> Solar_cell:Solar_Cell_Lightricity_S8040_CIC_Shorter_Tabs
Changed lines of the file:
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@@
 			)
 		)
-		(property "Footprint" "Solar_cell:Solar_Cell_Lightricity_S8040_CIC"
+		(property "Footprint" "Solar_cell:Solar_Cell_Lightricity_S8040_CIC_Shorter_Tabs"
 			(at 104.14 82.804 90)
 			(effects

Commit message: moved holes up 5mm, did what Jack said to do
Parts:
- Buck1: footprint Connection_Pads:2_Hirose_Pin -> Connection_Pads:DF13_Horizontal
Changed lines of the file:
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@@
 			)
 		)
-		(property "Footprint" "Connection_Pads:2_Hirose_Pin"
+		(property "Footprint" "Connection_Pads:DF13_Horizontal"
 			(at 123.19 83.82 0)
 			(effects

Commit message: changed ALOT of things, got it to a point to send mech models,solar panel harness on BS need changed
Connections:
- net at SC6.2 (-): now also Buck1.1 (BCR+); no longer Buck1.2 (BCR-)
- net at SC1.1 (+): now also Buck1.2 (BCR-); no longer Buck1.1 (BCR+)
Other:
- moved on the sheet: Buck1
Changed lines of the file:
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@@
-		)
-	)
-	(rectangle
-		(start 96.52 50.8)
-		(end 134.62 115.57)
-		(stroke
-			(width 0)
-			(type solid)
-		)
-		(fill
-			(type none)
 		)
 	)
@@
 	(wire
 		(pts
-			(xy 124.46 52.07) (xy 124.46 78.74)
+			(xy 125.73 52.07) (xy 125.73 81.28)
 		)
 		(stroke
@@
 	(wire
 		(pts
-			(xy 124.46 104.14) (xy 124.46 81.28)
+			(xy 125.73 81.28) (xy 124.46 81.28)
 		)
 		(stroke
@@
 	(wire
 		(pts
-			(xy 104.14 67.31) (xy 104.14 69.85)
+			(xy 125.73 104.14) (xy 125.73 83.82)
 		)
 		(stroke
@@
 	(wire
 		(pts
-			(xy 104.14 96.52) (xy 104.14 104.14)
+			(xy 125.73 83.82) (xy 124.46 83.82)
 		)
 		(stroke
@@
 	(wire
 		(pts
-			(xy 104.14 52.07) (xy 124.46 52.07)
+			(xy 104.14 67.31) (xy 104.14 69.85)
 		)
 		(stroke
@@
 	(wire
 		(pts
-			(xy 104.14 104.14) (xy 124.46 104.14)
+			(xy 104.14 96.52) (xy 104.14 104.14)
 		)
 		(stroke
@@
 	(wire
 		(pts
-			(xy 104.14 77.47) (xy 104.14 78.74)
+			(xy 104.14 52.07) (xy 125.73 52.07)
 		)
 		(stroke
@@
 		)
 	)
+	(wire
+		(pts
+			(xy 104.14 104.14) (xy 125.73 104.14)
+		)
+		(stroke
+			(width 0)
+			(type default)
+		)
+	)
+	(wire
+		(pts
+			(xy 104.14 77.47) (xy 104.14 78.74)
+		)
+		(stroke
+			(width 0)
+			(type default)
+		)
+	)
 	(symbol
 		(lib_id "Mechanical:MountingHole")
@@
 		(lib_name "Pad_1")
 		(lib_id "Connection_Pads:Pad")
-		(at 128.27 76.2 180)
+		(at 120.65 86.36 0)
 		(unit 1)
 		(exclude_from_sim no)
@@
 		(dnp no)
 		(property "Reference" "Solder_Pad3"
-			(at 127 76.8351 0)
+			(at 121.92 85.7249 0)
 			(effects
 				(font
@@
 		)
 		(property "Value" "~"
-			(at 128.27 73.66 0)
+			(at 120.65 88.9 0)
 			(effects
 				(font
@@
 		)
 		(property "Footprint" "Connection_Pads:Series_Connection_Pad"
-			(at 128.27 76.2 0)
+			(at 120.65 86.36 0)
 			(effects
 				(font
@@
 		)
 		(property "Datasheet" ""
-			(at 128.27 76.2 0)
+			(at 120.65 86.36 0)
 			(effects
 				(font
@@
 		)
 		(property "Description" ""
-			(at 128.27 76.2 0)
+			(at 120.65 86.36 0)
 			(effects
 				(font
@@
 	(symbol
 		(lib_id "Connection_Pads:Hirose_Connector")
-		(at 133.35 80.01 180)
+		(at 115.57 82.55 0)
 		(unit 1)
 		(exclude_from_sim no)
@@
 		(dnp no)
 		(property "Reference" "Hirose_Connector1"
-			(at 133.35 104.14 0)
+			(at 115.57 58.42 0)
 			(effects
 				(font
@@
 		)
 		(property "Value" "~"
-			(at 132.08 78.74 0)
+			(at 116.84 83.82 0)
 			(effects
 				(font
@@
 		)
 		(property "Footprint" "Connector_Hirose:Hirose_DF13-05P-1.25DSA_1x05_P1.25mm_Vertical"
-			(at 133.35 80.01 0)
+			(at 115.57 82.55 0)
 			(effects
 				(font
@@
 		)
 		(property "Datasheet" ""
-			(at 133.35 80.01 0)
+			(at 115.57 82.55 0)
 			(effects
 				(font
@@
 		)
 		(property "Description" ""
-			(at 133.35 80.01 0)
+			(at 115.57 82.55 0)
 			(effects
 				(font
@@
 	(symbol
 		(lib_id "Connection_Pads:Pad")
-		(at 133.35 80.01 180)
+		(at 115.57 82.55 0)
 		(unit 1)
 		(exclude_from_sim no)
@@
 		(fields_autoplaced yes)
 		(property "Reference" "Solder_Pad1"
-			(at 132.08 80.6451 0)
+			(at 116.84 81.9149 0)
 			(effects
 				(font
@@
 		)
 		(property "Value" "~"
-			(at 132.08 78.74 0)
+			(at 116.84 83.82 0)
 			(effects
 				(font
@@
 		)
 		(property "Footprint" ""
-			(at 133.35 80.01 0)
+			(at 115.57 82.55 0)
 			(effects
 				(font
@@
 		)
 		(property "Datasheet" ""
-			(at 133.35 80.01 0)
+			(at 115.57 82.55 0)
 			(effects
 				(font
@@
 		)
 		(property "Description" ""
-			(at 133.35 80.01 0)
+			(at 115.57 82.55 0)
 			(effects
 				(font
@@
 	(symbol
 		(lib_id "Connection_Pads:Pout_Hirose")
-		(at 123.19 83.82 180)
+		(at 125.73 78.74 0)
 		(unit 1)
 		(exclude_from_sim no)
@@
 		(dnp no)
 		(property "Reference" "Buck1"
-			(at 129.54 84.328 0)
+			(at 119.38 78.232 0)
 			(effects
 				(font
@@
 		)
 		(property "Value" "~"
-			(at 127 82.55 0)
+			(at 121.92 80.01 0)
 			(effects
 				(font
@@
 		)
 		(property "Footprint" "Connection_Pads:DF13_Horizontal"
-			(at 123.19 83.82 0)
+			(at 125.73 78.74 0)
 			(effects
 				(font
@@
 		)
 		(property "Datasheet" ""
-			(at 123.19 83.82 0)
+			(at 125.73 78.74 0)
 			(effects
 				(font
@@
 		)
 		(property "Description" ""
-			(at 123.19 83.82 0)
+			(at 125.73 78.74 0)
 			(effects
 				(font
@@
 	(symbol
 		(lib_id "Connection_Pads:Series_Connection")
-		(at 133.35 80.01 180)
+		(at 115.57 82.55 0)
 		(unit 1)
 		(exclude_from_sim no)
@@
 		(fields_autoplaced yes)
 		(property "Reference" "Connection1"
-			(at 132.08 80.6451 0)
+			(at 116.84 81.9149 0)
 			(effects
 				(font
@@
 		)
 		(property "Value" "~"
-			(at 132.08 78.74 0)
+			(at 116.84 83.82 0)
 			(effects
 				(font
@@
 		)
 		(property "Footprint" ""
-			(at 133.35 80.01 0)
+			(at 115.57 82.55 0)
 			(effects
 				(font
@@
 		)
 		(property "Datasheet" ""
-			(at 133.35 80.01 0)
+			(at 115.57 82.55 0)
 			(effects
 				(font
@@
 		)
 		(property "Description" ""
-			(at 133.35 80.01 0)
+			(at 115.57 82.55 0)
 			(effects
 				(font
@@
 		(lib_name "Pad_2")
 		(lib_id "Connection_Pads:Pad")
-		(at 133.35 80.01 180)
+		(at 115.57 82.55 0)
 		(unit 1)
 		(exclude_from_sim no)
@@
 		(fields_autoplaced yes)
 		(property "Reference" "Solder_Pad2"
-			(at 132.08 80.6451 0)
+			(at 116.84 81.9149 0)
 			(effects
 				(font
@@
 		)
 		(property "Value" "~"
-			(at 132.08 78.74 0)
+			(at 116.84 83.82 0)
 			(effects
 				(font
@@
 		)
 		(property "Footprint" "Connection_Pads:Series_Connection_Pad"
-			(at 133.35 80.01 0)
+			(at 115.57 82.55 0)
 			(effects
 				(font
@@
 		)
 		(property "Datasheet" ""
-			(at 133.35 80.01 0)
+			(at 115.57 82.55 0)
 			(effects
 				(font
@@
 		)
 		(property "Description" ""
-			(at 133.35 80.01 0)
-			(effects
-				(font
+			(at 115.57 82.55 0)
+			(effects
+				(font

Commit message: removed solder mask from footprint
Parts:
- SC3: footprint Solar_cell:Solar_Cell_Lightricity_S8040_CIC_Shorter_Tabs -> Solar_cell:Solar_Cell_Lightricity_S8040_CIC
Changed lines of the file:
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@@
 			)
 		)
-		(property "Footprint" "Solar_cell:Solar_Cell_Lightricity_S8040_CIC_Shorter_Tabs"
+		(property "Footprint" "Solar_cell:Solar_Cell_Lightricity_S8040_CIC"
 			(at 104.14 82.804 90)
 			(effects
