File: +x_panel/left-panel/left-panel.kicad_pcb (KiCad board)
At the start: 2 copper layers, 85 x 270 mm, 14 parts

Commit message: changed cover panels to have smaller power planes, also changed front panel DF13 from SMD to THT
Routing:
- net Net-(Buck1-BCR-): track 296.0 -> 293.1 mm
