File: Back_Blank_Face/Back_Blank_Face/Back_Blank_Face.kicad_sch (KiCad schematic)
At the start: 14 parts

Commit message: changed ALOT of things, got it to a point to send mech models,solar panel harness on BS need changed
Parts:
- added H15, H16, H17, H18, H19, H20, H21, H22: MountingHole, Small_Mounting_Holes:2.0mm_Mounting_Hole, symbol Mechanical:MountingHole

Commit message: Removed GND and PWR plane, replaced with traces, switches are now in series rather than in parallel
Parts:
- H19, H20, H21, H22: footprint Small_Mounting_Holes:2.0mm_Mounting_Hole -> MountingHole:MountingHole_2.5mm
Changed lines of the file:
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@@
 			)
 		)
-		(property "Footprint" "Small_Mounting_Holes:2.0mm_Mounting_Hole"
+		(property "Footprint" "MountingHole:MountingHole_2.5mm"
 			(at 204.47 99.06 0)
 			(effects
@@
 			)
 		)
-		(property "Footprint" "Small_Mounting_Holes:2.0mm_Mounting_Hole"
+		(property "Footprint" "MountingHole:MountingHole_2.5mm"
 			(at 204.47 88.9 0)
 			(effects
@@
 			)
 		)
-		(property "Footprint" "Small_Mounting_Holes:2.0mm_Mounting_Hole"
+		(property "Footprint" "MountingHole:MountingHole_2.5mm"
 			(at 203.2 69.85 0)
 			(effects
@@
 			)
 		)
-		(property "Footprint" "Small_Mounting_Holes:2.0mm_Mounting_Hole"
+		(property "Footprint" "MountingHole:MountingHole_2.5mm"
 			(at 204.47 80.01 0)
 			(effects
