File: Back_Blank_Face/Back_Blank_Face/Back_Blank_Face.kicad_pcb (KiCad board)
At the start: 2 copper layers, 87 x 326.5 mm, 18 parts

Commit message: added transceiver debug cutouts -Y face
Other:
- outline, holes or cut-outs redrawn
- board text added: "-Y"
- board text added: "5V USB CHARGE"
- board text added: "Battery Charging Port"
- board text added: "Compact Mag Harness Passthrough"
- board text added: "Debug"
- board text added: "OBC SD Boot"
- board text added: "OBC UART0 Serial"
- board text added: "OBC Umbilical Connector"
- board text added: "RBF Port"
- board text added: "Solar Panel Deployment ARM"
- board text added: "UHF"
- board text added: "UHF Antenna Deployment ARM"
- board text added: "VHF"
- board text added: "VHF Antenna Deployment ARM"
