File: front-panel/front-panel.kicad_pcb (KiCad board)
At the start: 2 copper layers, 87 x 326.5 mm, 7 parts

Commit message: Added projects for blank PCBs, updated solar panels
Parts:
- added H1: MountingHole, MountingHole:MountingHole_3.2mm_M3, F.Cu at (112.2, 259.9)
- added H10: MountingHole, MountingHole:MountingHole_2.7mm, F.Cu at (125.2, 35.9)
- added H11: MountingHole, MountingHole:MountingHole_2.7mm, F.Cu at (157.4, 35.9)
- added H12: MountingHole, MountingHole:MountingHole_2.7mm, F.Cu at (157.4, 14.7)
- added H13: MountingHole, MountingHole:MountingHole_3.2mm_M3, F.Cu at (188.2, 15.3)
- added H13: MountingHole, MountingHole:MountingHole_3.2mm_M3, F.Cu at (112.1, 15.3)
- added H2: MountingHole, MountingHole:MountingHole_3.2mm_M3, F.Cu at (112.1, 130.8)
- added H3: MountingHole, MountingHole:MountingHole_3.2mm_M3, F.Cu at (188.2, 259.8)
- added H4: MountingHole, MountingHole:MountingHole_3.2mm_M3, F.Cu at (188.2, 130.8)
- added H5: MountingHole, MountingHole:MountingHole_3.2mm_M3, F.Cu at (112.2, 306.9)
- added H6: MountingHole, MountingHole:MountingHole_3.2mm_M3, F.Cu at (188.2, -11.7)
- added H7: MountingHole, MountingHole:MountingHole_3.2mm_M3, F.Cu at (188.2, 306.9)
- added H8: MountingHole, MountingHole:MountingHole_3.2mm_M3, F.Cu at (112.1, -11.7)
- added H9: MountingHole, MountingHole:MountingHole_2.7mm, F.Cu at (125.2, 14.7)
- moved Buck2 63.6 mm to (178.7, 28.1), turned to 0 degrees
Routing:
- net Net-(Buck2-BCR-): track 259.4 -> 278.2 mm
- net Net-(Buck2-BCR+): track 68.5 -> 78.0 mm
Other:
- outline, holes or cut-outs redrawn

Commit message: Changes solar panels
Parts:
- moved SC14 4.00 mm to (134.4, 66.7)
Routing:
- net Net-(Buck2-BCR+): track 78.0 -> 8.04 mm, vias 1 -> 0
- net Net-(Buck2-BCR-): track 278.2 -> 281.3 mm
Changed lines of the file:
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@@
 	(footprint "Solar_cell:Solar_Cell_Lightricity_S8040_CIC_Shorter_Tabs"
 		(layer "F.Cu")
-		(at 134.4 70.65 -90)
+		(at 134.4 66.65 -90)
 		(property "Reference" "SC14"
 			(at 0 -0.5 270)
@@
 			(type solid)
 		)
+		(layer "F.SilkS")
+	)
+	(gr_circle
+		(center 125.15 35.92)
+		(end 125.15 33.68)
+		(stroke
+			(width 0.1)
+			(type solid)
+		)
+		(fill no)
 		(layer "F.SilkS")
 	)
@@
 	)
 	(segment
-		(start 148.315 41.185)
-		(end 164.31 41.185)
-		(width 4)
-		(layer "F.Cu")
-		(net 4)
-	)
-	(segment
-		(start 164.31 37.99)
-		(end 164.23 37.91)
-		(width 4)
-		(layer "F.Cu")
-		(net 4)
-	)
-	(segment
-		(start 168.835 41.185)
-		(end 168.895 41.245)
-		(width 4)
-		(layer "F.Cu")
-		(net 4)
-	)
-	(segment
-		(start 127.855 41.165)
-		(end 148.295 41.165)
-		(width 4)
-		(layer "F.Cu")
-		(net 4)
-	)
-	(segment
-		(start 164.31 41.185)
-		(end 168.835 41.185)
-		(width 4)
-		(layer "F.Cu")
-		(net 4)
-	)
-	(segment
-		(start 164.31 41.185)
-		(end 164.31 37.99)
-		(width 4)
-		(layer "F.Cu")
-		(net 4)
-	)
-	(segment
-		(start 168.895 41.245)
-		(end 182.6925 41.245)
-		(width 4)
-		(layer "F.Cu")
-		(net 4)
-	)
-	(segment
-		(start 182.6925 41.245)
-		(end 182.8175 41.12)
-		(width 4)
-		(layer "F.Cu")
-		(net 4)
-	)
-	(segment
-		(start 148.295 41.165)
-		(end 148.315 41.185)
-		(width 4)
-		(layer "F.Cu")
-		(net 4)
-	)
-	(via
-		(at 164.23 37.91)
-		(size 4)
-		(drill 3)
-		(layers "F.Cu" "B.Cu")
-		(net 4)
-	)
-	(segment
-		(start 164.23 37.91)
-		(end 164.25 37.89)
+		(start 168.2715 22.3285)
+		(end 170.5925 22.3285)
 		(width 4)
 		(layer "B.Cu")
@@
 	)
 	(segment
-		(start 168.2715 22.3285)
-		(end 170.5925 22.3285)
-		(width 4)
-		(layer "B.Cu")
-		(net 4)
-	)
-	(segment
 		(start 164.23 26.37)
 		(end 168.2715 22.3285)
-		(width 4)
-		(layer "B.Cu")
-		(net 4)
-	)
-	(segment
-		(start 164.23 37.91)
-		(end 164.23 26.37)
 		(width 4)
 		(layer "B.Cu")
@@
 	)
 	(segment
-		(start 175.2225 22.7325)
-		(end 174.8185 22.3285)
+		(start 178.97 264.81)
+		(end 178.97 26.48)
 		(width 4)
 		(layer "B.Cu")
@@
 	)
 	(segment
-		(start 173.83 269.95)
-		(end 175.2225 268.5575)
+		(start 174.8185 22.3285)
+		(end 174.7935 22.3285)
 		(width 4)
 		(layer "B.Cu")
@@
 	)
 	(segment
-		(start 174.8185 22.3285)
-		(end 174.7935 22.3285)
+		(start 178.97 26.48)
+		(end 174.8185 22.3285)
 		(width 4)
 		(layer "B.Cu")
@@
 	)
 	(segment
-		(start 175.2225 268.5575)
-		(end 175.2225 22.7325)
+		(start 173.83 269.95)
+		(end 178.97 264.81)
 		(width 4)
 		(layer "B.Cu")

Commit message: Updated panels based on dxf drawings from mech, need to move all holes up 5mm
Parts:
- moved Buck2 11.1 mm to (178.7, 39.2)
- moved H2 6.49 mm to (112.1, 124.3)
- moved H4 6.49 mm to (188.3, 124.3)
- moved H10 4.26 mm to (121.1, 37.0)
- moved H12 4.25 mm to (153.2, 15.7)
- moved H11 4.24 mm to (153.3, 36.9)
- moved H9 4.21 mm to (121.1, 15.8)
- moved SC7 3.75 mm to (108.2, 81.1)
- moved SC14 0.58 mm to (134.1, 67.1)
Routing:
- net Net-(SC14--): track 73.9 -> 16.2 mm
- net Net-(Buck2-BCR+): track 8.04 -> 40.0 mm, vias 0 -> 1
- net Net-(Buck2-BCR-): track 281.3 -> 273.6 mm
- added copper zone on B.Cu, net Net-(Buck2-BCR+)
- added copper zone on B.Cu, net Net-(Buck2-BCR-)
Other:
- outline, holes or cut-outs redrawn

Commit message: changed ALOT of things, got it to a point to send mech models,solar panel harness on BS need changed
Other:
- outline, holes or cut-outs redrawn
Changed lines of the file:
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@@
 		(tags "mountinghole M3")
 		(property "Reference" "H6"
-			(at 0 -4.15 0)
+			(at 0 4.38 0)
 			(layer "F.SilkS")
 			(effects
@@
 	)
 	(gr_line
-		(start 179.930046 9.33)
-		(end 165.93 9.33)
-		(stroke
-			(width 0.25)
-			(type default)
-		)
-		(locked yes)
-		(layer "Edge.Cuts")
-	)
-	(gr_rect
-		(start 165.753213 9.403176)
-		(end 180.106766 26.756747)
-		(stroke
-			(width 0.05)
-			(type default)
-		)
-		(fill no)
+		(start 179.930046 9.330001)
+		(end 165.9299 9.33)
+		(stroke
+			(width 0.25)
+			(type default)
+		)
 		(locked yes)
 		(layer "Edge.Cuts")
@@
 		(stroke
 			(width 0.25)
-			(type default)
-		)
-		(locked yes)
+			(type solid)
+		)
+		(locked yes)

Commit message: Rerouted some stuff
Routing:
- net Net-(SC14--): track 16.2 -> 87.5 mm
- net Net-(Buck2-BCR+): track 40.0 -> 72.9 mm
- net Net-(Buck2-BCR-): track 273.6 -> 282.0 mm
Changed lines of the file:
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@@
 			)
 		)
+		(sheetname "/")
+		(sheetfile "front-panel.kicad_sch")
 		(attr smd)
 		(fp_line
@@
 			)
 		)
+		(sheetname "/")
+		(sheetfile "front-panel.kicad_sch")
 		(attr smd)
 		(fp_line
@@
 			)
 		)
+		(sheetname "/")
+		(sheetfile "front-panel.kicad_sch")
 		(attr smd)
 		(fp_line
@@
 			)
 		)
+		(sheetname "/")
+		(sheetfile "front-panel.kicad_sch")
 		(attr smd)
 		(fp_line
@@
 			)
 		)
+		(sheetname "/")
+		(sheetfile "front-panel.kicad_sch")
 		(attr smd)
 		(fp_line
@@
 			)
 		)
+		(sheetname "/")
+		(sheetfile "front-panel.kicad_sch")
 		(attr smd)
 		(fp_line
@@
 			)
 		)
+		(sheetname "/")
+		(sheetfile "front-panel.kicad_sch")
 		(attr through_hole)
 		(fp_line
@@
 	)
 	(segment
+		(start 148.22 76.34)
+		(end 168.8 76.34)
+		(width 4)
+		(layer "F.Cu")
+		(net 3)
+	)
+	(segment
+		(start 148.22 76.34)
+		(end 127.835 76.34)
+		(width 4)
+		(layer "F.Cu")
+		(net 3)
+	)
+	(segment
 		(start 149.945 63.725)
-		(end 149.945 79.895)
+		(end 148.22 65.45)
+		(width 4)
+		(layer "F.Cu")
+		(net 3)
+	)
+	(segment
+		(start 148.22 65.45)
+		(end 148.22 76.34)
+		(width 4)
+		(layer "F.Cu")
+		(net 3)
+	)
+	(segment
+		(start 168.8 76.34)
+		(end 182.8375 76.34)
+		(width 4)
+		(layer "F.Cu")
+		(net 3)
+	)
+	(segment
+		(start 149.595 60.185)
+		(end 168.8 60.185)
 		(width 4)
 		(layer "F.Cu")
@@
 	)
 	(segment
-		(start 168.64 35.9)
+		(start 182.5925 35.9)
+		(end 168.64 35.9)
+		(width 4)
+		(layer "F.Cu")
+		(net 4)
+	)
+	(segment
+		(start 147.26 29.48)
+		(end 152.62 29.48)
+		(width 4)
+		(layer "F.Cu")
+		(net 4)
+	)
+	(segment
+		(start 152.62 29.48)
+		(end 162.1 29.48)
+		(width 4)
+		(layer "F.Cu")
+		(net 4)
+	)
+	(segment
+		(start 162.1 29.48)
 		(end 168.58 35.96)
 		(width 4)
@@
 	)
 	(segment
+		(start 151.945 29.48)
+		(end 152.62 29.48)
+		(width 4)
+		(layer "F.Cu")
+		(net 4)
+	)
+	(segment
 		(start 127.855 35.92)
 		(end 127.795 35.86)
@@
 	)
 	(segment
-		(start 182.5925 35.9)
-		(end 168.64 35.9)
+		(start 147.26 34.165)
+		(end 151.945 29.48)
+		(width 4)
+		(layer "F.Cu")
+		(net 4)
+	)
+	(segment
+		(start 147.26 35.92)
+		(end 147.26 34.165)
 		(width 4)
 		(layer "F.Cu")
@@
 	)
 	(segment
-		(start 160.445 283.135)
-		(end 174.7735 268.8065)
+		(start 149.515 283.135)
+		(end 174.7735 283.135)
 		(width 4)
 		(layer "F.Cu")
@@
 	)
 	(segment
-		(start 149.515 283.135)
-		(end 160.445 283.135)
+		(start 174.7735 283.135)
+		(end 174.7735 268.8065)
 		(width 4)
 		(layer "F.Cu")
@@
 			(thermal_gap 0.5)
 			(thermal_bridge_width 0.5)
+			(smoothing fillet)
+			(radius 1)
 		)
 		(polygon
 			(pts
-				(xy 172.86 27.37) (xy 177.26 27.39) (xy 177.26 34.05) (xy 176.2 37.11) (xy 173.33 37.21) (xy 172.87 34.03)
+				(xy 173.225 31.75) (xy 175 31.7575) (xy 176.775 31.765) (xy 176.775 39.175) (xy 172.775 39.175)
+				(xy 172.775 37.2) (xy 173.207469 34.80558) (xy 173.219606 34.658928) (xy 173.225 34.528349) (xy 173.225 34.2)
 			)
 		)
@@
 			(thermal_gap 0.5)
 			(thermal_bridge_width 0.5)
+			(smoothing fillet)
+			(radius 1)
 		)
 		(polygon

Commit message: reviewed boards
Changed lines of the file:
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@@
 		)
 		(fp_line
-			(start -10.45 33.1)
-			(end 3.55 47.35)
-			(stroke
-				(width 0.1)
-				(type solid)
-			)
-			(layer "F.CrtYd")
-		)
-		(fp_line
 			(start -10.43 33.03)
 			(end 3.57 47.28)
@@
 		)
 		(fp_line
-			(start -10.45 33.1)
-			(end 3.55 47.35)
-			(stroke
-				(width 0.1)
-				(type solid)
-			)
-			(layer "F.CrtYd")
-		)
-		(fp_line
 			(start -10.43 33.03)
 			(end 3.57 47.28)
@@
 		(sheetfile "front-panel.kicad_sch")
 		(attr smd)
+		(fp_poly
+			(pts
+				(xy -26.655 12.105) (xy -12.66 12.105) (xy -12.66 26.057802)
+			)
+			(stroke
+				(width 0)
+				(type solid)
+			)
+			(fill yes)
+			(layer "F.Mask")
+		)
 		(fp_line
 			(start -12.74 26.17)
@@
 			)
 		)
+		(pad "" smd rect
+			(at -19.6575 -20.815)
+			(size 65.84 13.995)
+			(layers "F.Mask")
+		)
+		(pad "" smd rect
+			(at 0.2375 -13.838599)
+			(size 79.792802 25.795)
+			(layers "F.Mask")
+		)
 		(pad "1" smd rect
 			(at -31.3 -12.915 270)
@@
 		)
 		(pad "2" smd roundrect
-			(at -6.925 -15.545 270)
+			(at -6.93 -15.54 270)
 			(size 16.17 57.37)
 			(layers "F.Cu" "F.Mask" "F.Paste")
@@
 			(pinfunction "-")
 			(pintype "passive")
-			(clearance 0)
 		)
 		(embedded_fonts no)
@@
 	)
 	(zone
-		(net 0)
-		(net_name "")
-		(layer "F.Mask")
-		(hatch edge 0.5)
-		(connect_pads
-			(clearance 0.5)
-		)
-		(min_thickness 0.25)
-		(filled_areas_thickness no)
-		(fill yes
-			(thermal_gap 0.5)
-			(thermal_bridge_width 0.5)
-		)
-		(polygon
-			(pts
-				(xy 107.89 80.36) (xy 107.89 54.36) (xy 121.89 40.36) (xy 187.88 40.37) (xy 187.88 80.37)
-			)
-		)
-	)
-	(zone

Commit message: Removed GND and PWR plane, replaced with traces, switches are now in series rather than in parallel
Parts:
- added H15: MountingHole, MountingHole:MountingHole_2.5mm, F.Cu at (155.2, 0.35)
- added H16: MountingHole, MountingHole:MountingHole_2.5mm, F.Cu at (155.2, 22.3)
- added H17: MountingHole, MountingHole:MountingHole_2.5mm, F.Cu at (177.2, 22.3)
- added H18: MountingHole, MountingHole:MountingHole_2.5mm, F.Cu at (177.2, 0.33)
- H10, H11, H12, H9: footprint MountingHole:MountingHole_2.7mm -> MountingHole:MountingHole_2.5mm
- moved Buck2 47.7 mm to (132.2, 28.6), turned to 180 degrees
- moved H11 41.0 mm to (145.1, -3.28)
- moved H12 32.2 mm to (123.9, 28.9)
- moved H10 25.3 mm to (145.1, 28.9)
- moved H9 19.2 mm to (123.9, -3.26)
- moved SC8 1.00 mm to (154.4, 143.3)
- moved SC9 0.75 mm to (107.6, 174.4)
- moved SC10 0.59 mm to (107.5, 215.4)
- moved SC7 0.39 mm to (107.8, 81.0)
- moved SC14 0.13 mm to (134.0, 67.0)
Routing:
- net Net-(Buck2-BCR-): track 282.0 -> 302.3 mm
- net Net-(Buck2-BCR+): track 72.9 -> 55.9 mm
Other:
- outline, holes or cut-outs redrawn
