File: front-panel/front-panel.kicad_pcb (KiCad board)
At the start: 2 copper layers, 87 x 326.5 mm, 25 parts

Commit message: added transceiver debug cutouts -Y face
Parts:
- moved Buck2 21.1 mm to (159.7, 37.2)
Routing:
- net Net-(Buck2-BCR-): track 302.4 -> 319.3 mm
- net Net-(Buck2-BCR+): track 68.5 -> 56.5 mm
Other:
- board text added: "+Y"
Changed lines of the file:
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@@
 			(drillshape 0)
 			(scaleselection 1)
-			(outputdirectory "../../Board_Order_GRB/Front-Panel/")
+			(outputdirectory "../../Board_Order_3/plus_y_panel/")
 		)
 	)
@@
 	(footprint "Connection_Pads:Hirose_DF13-02P-1.25DSA_1x02_P1.25mm_Vertical"
 		(layer "B.Cu")
-		(at 138.615 36.77 180)
+		(at 159.68 37.18 180)
 		(descr "Hirose DF13 through hole, DF13-02P-1.25DSA, 2 Pins per row (https://www.hirose.com/product/en/products/DF13/DF13-2P-1.25DSA%2850%29/)")
 		(tags "connector Hirose DF13 vertical")
@@
 		(layer "Edge.Cuts")
 	)
+	(gr_text "+Y"
+		(at 132.21 -3.51 0)
+		(layer "F.SilkS")
+		(effects
+			(font
+				(size 10 10)
+				(thickness 1)
+			)
+			(justify left bottom)
+		)
+	)
 	(dimension
 		(type orthogonal)
@@
 	)
 	(segment
-		(start 124.63 272.67)
-		(end 124.63 41.55)
+		(start 154.49 37.05)
+		(end 154.57 36.97)
 		(width 4)
 		(layer "B.Cu")
@@
 	)
 	(segment
-		(start 124.63 41.55)
-		(end 129.54 36.64)
+		(start 124.63 272.67)
+		(end 124.63 48.98)
 		(width 4)
 		(layer "B.Cu")
@@
 	)
 	(segment
-		(start 129.54 36.64)
-		(end 133.17 36.64)
+		(start 136.56 37.05)
+		(end 154.49 37.05)
 		(width 4)
 		(layer "B.Cu")
@@
 	)
 	(segment
-		(start 158.8 35.96)
-		(end 153.26 35.96)
+		(start 124.63 48.98)
+		(end 136.56 37.05)
 		(width 4)
-		(layer "F.Cu")
-		(net "Net-(Buck2-BCR+)")
+		(layer "B.Cu")
+		(net "Net-(Buck2-BCR-)")
 	)
 	(segment
@@
 	)
 	(segment
-		(start 146.684118 34.21)
-		(end 129.126107 34.21)
+		(start 148.127615 35.653497)
+		(end 146.684118 34.21)
 		(width 3)
 		(layer "F.Cu")
@@
 	)
 	(segment
-		(start 153.26 35.96)
-		(end 168.58 35.96)
-		(width 4)
+		(start 127.68261 35.653497)
+		(end 127.600269 35.735838)
+		(width 3)
 		(layer "F.Cu")
 		(net "Net-(Buck2-BCR+)")
 	)
 	(segment
-		(start 148.127615 35.653497)
-		(end 146.684118 34.21)
-		(width 3)
+		(start 147.115 35.96)
+		(end 146.965 35.81)
+		(width 4)
 		(layer "F.Cu")
 		(net "Net-(Buck2-BCR+)")
 	)
 	(segment
-		(start 158.8 35.96)
-		(end 147.115 35.96)
-		(width 4)
+		(start 148.127615 35.653497)
+		(end 127.68261 35.653497)
+		(width 3)
 		(layer "F.Cu")
 		(net "Net-(Buck2-BCR+)")
 	)
 	(segment
-		(start 147.115 35.96)
-		(end 146.965 35.81)
-		(width 4)
+		(start 167.61 34.01)
+		(end 150.051989 34.01)
+		(width 3)
 		(layer "F.Cu")
 		(net "Net-(Buck2-BCR+)")
@@
 	)
 	(via
-		(at 158.8 35.96)
+		(at 176.1 35.9)
 		(size 4)
 		(drill 3)
@@
 		(polygon
 			(pts
-				(xy 137.930218 34.92) (xy 137.922718 36.695) (xy 137.915218 38.47) (xy 130.205218 38.47) (xy 130.205218 34.65)
-				(xy 133.47681 34.65) (xy 134.874638 34.902469) (xy 135.02129 34.914606) (xy 135.151869 34.92) (xy 135.480218 34.92)
+				(xy 158.951821 35.274389) (xy 158.933741 37.024181) (xy 158.926239 38.8) (xy 151.316356 38.8) (xy 151.316356 34.98)
+				(xy 154.587948 34.98) (xy 155.985776 35.232469) (xy 156.132428 35.244606) (xy 156.263007 35.25)
+				(xy 156.591356 35.25)
 			)
 		)
@@
 		(polygon
 			(pts
-				(xy 161.233213 33.502101) (xy 161.192593 38.7293) (xy 141.98 38.58) (xy 138.17 38.63) (xy 138.24 34.93)
+				(xy 179.133501 33.30479) (xy 179.1265 38.974541) (xy 163.1 38.85) (xy 159.174971 38.90151) (xy 159.244865 35.20715)
 			)
 		)
