File: -z_blank_face/-z_blank_face/-z_blank_face.kicad_sch (KiCad schematic)
At the start: 0 parts

Commit message: changed cover panels to have smaller power planes, also changed front panel DF13 from SMD to THT
Parts:
- added H1, H2, H3, H4, H5, H6, H7, H8: MountingHole, MountingHole:MountingHole_2.7mm, symbol Mechanical:MountingHole
